File: RFM69-Gateway-logger.brd (EAGLE design)
At the start: 40 x 40 mm, 34 parts, among them IC3 MCP1703-3.3V, J3 MicroUSB (5V), U1 RFM69HCW, U2 ATMEGA328P-MU, X1 16 MHz

Commit message: Adjusted antenna & silkscreen
Parts:
- moved U$6 15.2 mm to (1.63, 33.9)
Routing:
- net ANA: track 8.78 -> 6.46 mm
Changed lines of the file:
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@@
 <layer number="47" name="Measures" color="7" fill="1" visible="no" active="yes"/>
 <layer number="48" name="Document" color="7" fill="1" visible="no" active="yes"/>
-<layer number="49" name="Reference" color="7" fill="1" visible="yes" active="yes"/>
+<layer number="49" name="Reference" color="7" fill="1" visible="no" active="yes"/>
 <layer number="50" name="dxf" color="7" fill="1" visible="no" active="yes"/>
 <layer number="51" name="tDocu" color="6" fill="1" visible="no" active="yes"/>
@@
 <layer number="116" name="Patch_BOT" color="9" fill="4" visible="no" active="yes"/>
 <layer number="118" name="Rect_Pads" color="7" fill="1" visible="no" active="yes"/>
-<layer number="121" name="_tsilk" color="7" fill="1" visible="yes" active="yes"/>
+<layer number="121" name="_tsilk" color="25" fill="1" visible="yes" active="yes"/>
 <layer number="122" name="_bsilk" color="12" fill="1" visible="yes" active="yes"/>
 <layer number="123" name="tTestmark" color="7" fill="1" visible="no" active="yes"/>
@@
 <attribute name="MPN" value="RFM69HW" x="8.6016" y="19.9956" size="1.778" layer="28" rot="MR90" display="off"/>
 <attribute name="PROD_ID" value="IC-11997, IC-12053" x="8.6016" y="19.9956" size="1.778" layer="28" rot="MR90" display="off"/>
-<attribute name="VALUE" x="17.8148" y="18.2124" size="0.6096" layer="122" font="vector" rot="MR270" align="bottom-right"/>
-</element>
-<element name="U$6" library="LowPowerLab" package="RFM12B-ANTENNA" value="RFM12B_ANTENNA" x="1.5268" y="18.7466"/>
+<attribute name="VALUE" x="17.8148" y="18.2124" size="0.6096" layer="121" font="vector" rot="MR270" align="bottom-right"/>
+</element>
+<element name="U$6" library="LowPowerLab" package="RFM12B-ANTENNA" value="RFM12B_ANTENNA" x="1.6268" y="33.9466"/>
 <element name="JP1" library="SparkFun-Connectors" package="MICRO-SD-SOCKET-PP" value="MicroSD socket" x="19.9848" y="15.4748" smashed="yes" rot="R180">
 <attribute name="PROD_ID" value="CONN-07820" x="19.9848" y="15.4748" size="1.778" layer="27" rot="R180" display="off"/>
-<attribute name="VALUE" x="33.9748" y="16.9948" size="0.6096" layer="27" font="vector" rot="R180"/>
+<attribute name="VALUE" x="33.9748" y="16.9948" size="0.6096" layer="121" font="vector" rot="R180"/>
 </element>
 <element name="DS3234" library="SparkFun-FreqCtrl" package="DS3234" value="DS3234" x="11.2568" y="8.67" smashed="yes" rot="R90">
 <attribute name="MPN" value="DS3234S#" x="11.2568" y="8.67" size="1.778" layer="27" rot="R90" display="off"/>
-<attribute name="NAME" x="13.2618" y="1.385" size="0.6096" layer="27" font="vector" rot="R180"/>
+<attribute name="NAME" x="13.2618" y="1.385" size="0.6096" layer="121" font="vector" rot="R180"/>
 </element>
 <element name="BAT1" library="SparkFun-Electromechanical" package="BATTCON_12MM" value="" x="5.768" y="26.2992" rot="R90">
@@
 </element>
 <element name="R13" library="adafruit" library_urn="urn:adsk.eagle:library:420" package="R0402" value="10K" x="35.3388" y="5.8672" smashed="yes" rot="R270">
-<attribute name="VALUE" x="36.4068" y="6.8022" size="0.6096" layer="27" font="vector" rot="R270"/>
+<attribute name="VALUE" x="36.4068" y="6.8022" size="0.6096" layer="121" font="vector" rot="R270"/>
 </element>
 <element name="C15" library="adafruit" library_urn="urn:adsk.eagle:library:420" package="C0402" value="1uF" x="35.3088" y="12.9328" smashed="yes" rot="R90">
-<attribute name="VALUE" x="36.9138" y="12.0978" size="0.6096" layer="27" font="vector" rot="R90"/>
+<attribute name="VALUE" x="36.9138" y="12.0978" size="0.6096" layer="121" font="vector" rot="R90"/>
 </element>
 <element name="R8" library="adafruit" library_urn="urn:adsk.eagle:library:420" package="R0402" value="10K" x="17.8372" y="1.2088" smashed="yes" rot="R180">
-<attribute name="VALUE" x="18.6722" y="2.4408" size="0.6096" layer="27" font="vector" rot="R180"/>
+<attribute name="VALUE" x="18.6722" y="2.4408" size="0.6096" layer="121" font="vector" rot="R180"/>
 </element>
 <element name="C3" library="adafruit" library_urn="urn:adsk.eagle:library:420" package="C0402" value="22pF" x="18.5088" y="7.4004" smashed="yes" rot="R90">
-<attribute name="VALUE" x="17.4654" y="8.9862" size="0.6096" layer="27" font="vector"/>
+<attribute name="VALUE" x="17.4654" y="8.9862" size="0.6096" layer="121" font="vector"/>
 </element>
 <element name="J3" library="SparkFun-Connectors" package="USB-MICROB" value="MicroUSB (5V)" x="20.0036" y="38.9952" smashed="yes" rot="R180">
@@
 </element>
 <element name="C7" library="adafruit" library_urn="urn:adsk.eagle:library:420" package="C0402" value="0.1uF" x="24.7" y="20.3" smashed="yes" rot="R90">
-<attribute name="VALUE" x="26.305" y="19.165" size="0.6096" layer="27" font="vector" rot="R90"/>
+<attribute name="VALUE" x="26.305" y="19.165" size="0.6096" layer="121" font="vector" rot="R90"/>
 </element>
 <element name="C5" library="adafruit" library_urn="urn:adsk.eagle:library:420" package="C0402" value="0.1uF" x="27.5" y="24.1" smashed="yes">
-<attribute name="VALUE" x="26.465" y="24.795" size="0.6096" layer="27" font="vector"/>
+<attribute name="VALUE" x="26.465" y="24.795" size="0.6096" layer="121" font="vector"/>
 </element>
 <element name="R3" library="adafruit" library_urn="urn:adsk.eagle:library:420" package="R0402" value="27" x="18.7" y="33.6" smashed="yes" rot="R180">
-<attribute name="VALUE" x="19.435" y="34.932" size="0.6096" layer="27" font="vector" rot="R180"/>
+<attribute name="VALUE" x="19.435" y="34.932" size="0.6096" layer="121" font="vector" rot="R180"/>
 </element>
 <element name="R5" library="adafruit" library_urn="urn:adsk.eagle:library:420" package="R0402" value="27" x="21.3" y="33.6" smashed="yes">
-<attribute name="VALUE" x="20.965" y="34.368" size="0.6096" layer="27" font="vector"/>
+<attribute name="VALUE" x="20.965" y="34.368" size="0.6096" layer="121" font="vector"/>
 </element>
 <element name="R4" library="adafruit" library_urn="urn:adsk.eagle:library:420" package="R0402" value="47" x="11.7" y="37.1" smashed="yes" rot="R180">
-<attribute name="VALUE" x="11.735" y="36.332" size="0.6096" layer="27" font="vector" rot="R180"/>
+<attribute name="VALUE" x="11.735" y="36.332" size="0.6096" layer="121" font="vector" rot="R180"/>
 </element>
 <element name="R6" library="adafruit" library_urn="urn:adsk.eagle:library:420" package="R0402" value="47" x="8.2" y="37.1" smashed="yes">
-<attribute name="VALUE" x="8.265" y="35.768" size="0.6096" layer="27" font="vector"/>
+<attribute name="VALUE" x="8.265" y="35.768" size="0.6096" layer="121" font="vector"/>
 </element>
 <element name="D2" library="Adafruit Feather 32u4 Bluefruit LE" package="MICROBUILDER_SOD-123" value="" x="29.6" y="36.4" smashed="yes" rot="R180">
-<attribute name="NAME" x="33.77" y="36.684" size="0.6096" layer="27" font="vector" rot="R180"/>
+<attribute name="NAME" x="33.77" y="36.684" size="0.6096" layer="121" font="vector" rot="R180"/>
 <attribute name="VALUE" x="30.87" y="38.178" size="0.4064" layer="27" ratio="10" rot="R180"/>
 </element>
@@
 <element name="U$8" library="ADS1x15" package="MOUNTINGHOLE_2.0_PLATED" value="MOUNTINGHOLE2.0" x="2.5" y="2.5"/>
 <element name="R7" library="adafruit" library_urn="urn:adsk.eagle:library:420" package="R0402" value="10K" x="27.5" y="26.7" smashed="yes">
-<attribute name="VALUE" x="26.765" y="27.568" size="0.6096" layer="27" font="vector"/>
+<attribute name="VALUE" x="26.765" y="27.568" size="0.6096" layer="121" font="vector"/>
 </element>
 <element name="R1" library="adafruit" library_urn="urn:adsk.eagle:library:420" package="R0402" value="10K" x="9.7" y="17.9" smashed="yes">
-<attribute name="VALUE" x="9.065" y="18.768" size="0.6096" layer="27" font="vector"/>
+<attribute name="VALUE" x="9.065" y="18.768" size="0.6096" layer="121" font="vector"/>
 </element>
 </elements>
@@
 <contactref element="U1" pad="9"/>
 <contactref element="U$6" pad="P$1"/>
-<wire x1="1.6016" y1="27.4956" x2="1.6016" y2="18.8214" width="1.016" layer="16"/>
-<wire x1="1.6016" y1="18.8214" x2="1.5268" y2="18.7466" width="1.016" layer="16"/>
+<wire x1="1.6016" y1="27.4956" x2="1.6016" y2="33.9214" width="1.016" layer="16"/>
+<wire x1="1.6016" y1="33.9214" x2="1.6268" y2="33.9466" width="1.016" layer="16"/>
 </signal>
 <signal name="N$3">

Commit message: Minor adjustments
Routing:
- net N$7: track 15.1 -> 17.4 mm
Changed lines of the file:
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@@
 <text x="38.658" y="19.9697" size="0.8128" layer="22" font="vector" ratio="9" rot="SMR270" align="bottom-center">v0.1   2017</text>
 <text x="39.1993" y="19.9951" size="0.6604" layer="21" font="vector" ratio="7" rot="R90" align="bottom-center">RFM69 Gateway logger</text>
-<text x="0.8807" y="17.0105" size="0.508" layer="21" font="vector">ANT</text>
+<text x="3.2895" y="33.4807" size="0.508" layer="21" font="vector" rot="R90">ANT</text>
 <wire x1="0" y1="2.5" x2="0" y2="37.5" width="0" layer="20"/>
 <wire x1="2.5" y1="40" x2="37.5" y2="40" width="0" layer="20"/>
@@
 </element>
 <element name="R8" library="adafruit" library_urn="urn:adsk.eagle:library:420" package="R0402" value="10K" x="17.8372" y="1.2088" smashed="yes" rot="R180">
-<attribute name="VALUE" x="18.6722" y="2.4408" size="0.6096" layer="121" font="vector" rot="R180"/>
+<attribute name="VALUE" x="14.9278" y="0.8592" size="0.6096" layer="121" font="vector"/>
 </element>
 <element name="C3" library="adafruit" library_urn="urn:adsk.eagle:library:420" package="C0402" value="22pF" x="18.5088" y="7.4004" smashed="yes" rot="R90">
-<attribute name="VALUE" x="17.4654" y="8.9862" size="0.6096" layer="121" font="vector"/>
+<attribute name="VALUE" x="18.0862" y="11.3346" size="0.6096" layer="121" font="vector" rot="R270"/>
 </element>
 <element name="J3" library="SparkFun-Connectors" package="USB-MICROB" value="MicroUSB (5V)" x="20.0036" y="38.9952" smashed="yes" rot="R180">
@@
 </element>
 <element name="R3" library="adafruit" library_urn="urn:adsk.eagle:library:420" package="R0402" value="27" x="18.7" y="33.6" smashed="yes" rot="R180">
-<attribute name="VALUE" x="19.435" y="34.932" size="0.6096" layer="121" font="vector" rot="R180"/>
+<attribute name="VALUE" x="19.205" y="32.802" size="0.6096" layer="121" font="vector" rot="R180"/>
 </element>
 <element name="R5" library="adafruit" library_urn="urn:adsk.eagle:library:420" package="R0402" value="27" x="21.3" y="33.6" smashed="yes">
-<attribute name="VALUE" x="20.965" y="34.368" size="0.6096" layer="121" font="vector"/>
+<attribute name="VALUE" x="20.795" y="32.198" size="0.6096" layer="121" font="vector"/>
 </element>
 <element name="R4" library="adafruit" library_urn="urn:adsk.eagle:library:420" package="R0402" value="47" x="11.7" y="37.1" smashed="yes" rot="R180">
@@
 <contactref element="TX" pad="MINUS"/>
 <contactref element="FT231XQ-R" pad="CBUS2"/>
-<wire x1="20.4344" y1="30.5348" x2="20.4344" y2="31.6344" width="0.254" layer="1"/>
-<wire x1="20.4344" y1="31.6344" x2="20.9" y2="32.1" width="0.254" layer="1"/>
-<via x="20.9" y="32.1" extent="1-16" drill="0.35" diameter="0.127"/>
-<wire x1="16.5" y1="32.1" x2="20.9" y2="32.1" width="0.254" layer="16"/>
+<via x="22" y="32.1" extent="1-16" drill="0.35" diameter="0.127"/>
+<wire x1="16.5" y1="32.1" x2="22" y2="32.1" width="0.254" layer="16"/>
 <via x="14.2" y="38.2" extent="1-16" drill="0.35" diameter="0.127"/>
 <wire x1="14.2" y1="38.2" x2="14.2" y2="38.6" width="0.254" layer="1"/>
@@
 <wire x1="14.2" y1="38.2" x2="14.2" y2="34.4" width="0.254" layer="16"/>
 <wire x1="14.2" y1="34.4" x2="16.5" y2="32.1" width="0.254" layer="16"/>
+<wire x1="20.4344" y1="31.7344" x2="20.8" y2="32.1" width="0.254" layer="1"/>
+<wire x1="20.8" y1="32.1" x2="22" y2="32.1" width="0.254" layer="1"/>
+<wire x1="20.4344" y1="30.5348" x2="20.4344" y2="31.7344" width="0.254" layer="1"/>
 </signal>
 <signal name="N$8">
@@
 <wire x1="25" y1="29" x2="25" y2="30.8" width="0.254" layer="1"/>
 <wire x1="25" y1="30.8" x2="24.9" y2="30.8" width="0.254" layer="16"/>
-<wire x1="24.9" y1="30.8" x2="24.2" y2="31.5" width="0.254" layer="16"/>
-<wire x1="22.2" y1="31.5" x2="24.2" y2="31.5" width="0.254" layer="16"/>
-<wire x1="16.9" y1="30.9" x2="21.6" y2="30.9" width="0.254" layer="16"/>
-<wire x1="21.6" y1="30.9" x2="22.2" y2="31.5" width="0.254" layer="16"/>
+<wire x1="24.2" y1="31.5" x2="24.9" y2="30.8" width="0.254" layer="16"/>
+<wire x1="22.4" y1="30.9" x2="23" y2="31.5" width="0.254" layer="16"/>
+<wire x1="23" y1="31.5" x2="24.2" y2="31.5" width="0.254" layer="16"/>
+<wire x1="16.9" y1="30.9" x2="22.4" y2="30.9" width="0.254" layer="16"/>
 </signal>
 <signal name="DTR">
