File: RFM69-Gateway-logger.brd (EAGLE design)
At the start: 40 x 40 mm, 34 parts, among them IC3 MCP1703-3.3V, J3 MicroUSB (5V), U1 RFM69HCW, U2 ATMEGA328P-MU, X1 16 MHz

Commit message: ANT pad adjusted
some GND pours adjusted
Parts:
- moved U$6 28.0 mm to (1.53, 5.95)
Routing:
- net ANA: track 6.46 -> 21.6 mm, vias 0 -> 1
- net N$3: track 16.3 -> 12.9 mm
- net GND: vias 9 -> 12
Changed lines of the file:
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@@
 <setting verticaltext="up"/>
 </settings>
-<grid distance="3.93700787" unitdist="mil" unit="mil" style="lines" multiple="1" display="yes" altdistance="0.01" altunitdist="mm" altunit="mm"/>
+<grid distance="2" unitdist="mil" unit="mil" style="lines" multiple="1" display="yes" altdistance="0.01" altunitdist="mm" altunit="mm"/>
 <layers>
 <layer number="1" name="Top" color="4" fill="1" visible="yes" active="yes"/>
@@
 <layer number="118" name="Rect_Pads" color="7" fill="1" visible="no" active="yes"/>
 <layer number="121" name="_tsilk" color="25" fill="1" visible="yes" active="yes"/>
-<layer number="122" name="_bsilk" color="12" fill="1" visible="yes" active="yes"/>
+<layer number="122" name="_bsilk" color="24" fill="1" visible="yes" active="yes"/>
 <layer number="123" name="tTestmark" color="7" fill="1" visible="no" active="yes"/>
 <layer number="124" name="bTestmark" color="7" fill="1" visible="no" active="yes"/>
@@
 <text x="38.658" y="19.9697" size="0.8128" layer="22" font="vector" ratio="9" rot="SMR270" align="bottom-center">v0.1   2017</text>
 <text x="39.1993" y="19.9951" size="0.6604" layer="21" font="vector" ratio="7" rot="R90" align="bottom-center">RFM69 Gateway logger</text>
-<text x="3.2895" y="33.4807" size="0.508" layer="21" font="vector" rot="R90">ANT</text>
+<text x="2.7557" y="6.5497" size="0.508" layer="21" font="vector" rot="SR270">ANT</text>
 <wire x1="0" y1="2.5" x2="0" y2="37.5" width="0" layer="20"/>
 <wire x1="2.5" y1="40" x2="37.5" y2="40" width="0" layer="20"/>
@@
 <attribute name="MPN" value="RFM69HW" x="8.6016" y="19.9956" size="1.778" layer="28" rot="MR90" display="off"/>
 <attribute name="PROD_ID" value="IC-11997, IC-12053" x="8.6016" y="19.9956" size="1.778" layer="28" rot="MR90" display="off"/>
-<attribute name="VALUE" x="1.7148" y="18.7124" size="0.6096" layer="122" font="vector" rot="MR270" align="bottom-right"/>
-</element>
-<element name="U$6" library="LowPowerLab" package="RFM12B-ANTENNA" value="RFM12B_ANTENNA" x="1.6268" y="33.9466"/>
+<attribute name="VALUE" x="10.9876" y="30.5148" size="0.6096" layer="122" font="vector" rot="MR180" align="bottom-right"/>
+</element>
+<element name="U$6" library="LowPowerLab" package="RFM12B-ANTENNA" value="RFM12B_ANTENNA" x="1.5268" y="5.9466"/>
 <element name="JP1" library="SparkFun-Connectors" package="MICRO-SD-SOCKET-PP" value="MicroSD socket" x="19.9848" y="15.4748" smashed="yes" rot="R180">
 <attribute name="PROD_ID" value="CONN-07820" x="19.9848" y="15.4748" size="1.778" layer="27" rot="R180" display="off"/>
@@
 <via x="31" y="14.4" extent="1-16" drill="0.35" diameter="0.127"/>
 <via x="12.1" y="19" extent="1-16" drill="0.35" diameter="0.127"/>
-<via x="13.8" y="3.3" extent="1-16" drill="0.35" diameter="0.127"/>
 <via x="18.7" y="14.3" extent="1-16" drill="0.35" diameter="0.127"/>
 <via x="31.5" y="26.1" extent="1-16" drill="0.35" diameter="0.127"/>
@@
 <wire x1="17.7024" y1="20.6548" x2="19.7548" y2="20.6548" width="0.254" layer="1"/>
 <wire x1="19.7548" y1="20.6548" x2="20" y2="20.9" width="0.254" layer="1"/>
+<via x="3.3076" y="7.6452" extent="1-16" drill="0.35" diameter="0.127"/>
+<via x="5.5936" y="1.5492" extent="1-16" drill="0.35" diameter="0.127"/>
+<via x="3.1044" y="17.3988" extent="1-16" drill="0.35" diameter="0.127"/>
+<via x="1.5804" y="34.0104" extent="1-16" drill="0.35" diameter="0.127"/>
 </signal>
 <signal name="D10_SS">
@@
 <wire x1="21.2524" y1="17.1476" x2="21.6" y2="16.8" width="0.254" layer="1"/>
 <via x="21.6" y="16.8" extent="1-16" drill="0.35" diameter="0.127"/>
-<via x="26.2" y="7.7" extent="1-16" drill="0.35" diameter="0.127"/>
+<via x="25.5396" y="8.3096" extent="1-16" drill="0.35" diameter="0.127"/>
 <wire x1="26.7248" y1="7.1752" x2="26.7248" y2="4.7748" width="0.254" layer="1"/>
-<wire x1="26.7248" y1="7.1752" x2="26.2" y2="7.7" width="0.254" layer="1"/>
+<wire x1="26.7248" y1="7.1752" x2="25.5396" y2="8.3096" width="0.254" layer="1"/>
 <wire x1="6.5718" y1="6.765" x2="10.035" y2="6.765" width="0.254" layer="1"/>
 <wire x1="10.035" y1="6.765" x2="10.65" y2="6.15" width="0.254" layer="1"/>
@@
 <via x="10.65" y="6.15" extent="1-16" drill="0.35" diameter="0.127"/>
 <wire x1="21.6" y1="16.8" x2="21.6" y2="12.3" width="0.254" layer="16"/>
-<wire x1="21.6" y1="12.3" x2="26.2" y2="7.7" width="0.254" layer="16"/>
+<wire x1="21.6" y1="12.3" x2="25.5396" y2="8.3096" width="0.254" layer="16"/>
 </signal>
 <signal name="D12_MISO">
@@
 <wire x1="9.6016" y1="8.6016" x2="8.7" y2="7.7" width="0.254" layer="16"/>
 <wire x1="24.5248" y1="4.7748" x2="24.5248" y2="2.9248" width="0.254" layer="1"/>
-<wire x1="24.5248" y1="2.9248" x2="23.9" y2="2.3" width="0.254" layer="1"/>
-<via x="23.9" y="2.3" extent="1-16" drill="0.35" diameter="0.127"/>
-<wire x1="23.9" y1="2.3" x2="13.4" y2="2.3" width="0.254" layer="16"/>
-<wire x1="13.4" y1="2.3" x2="12.4" y2="3.3" width="0.254" layer="16"/>
+<via x="23.646" y="2.046" extent="1-16" drill="0.35" diameter="0.127"/>
+<wire x1="23.646" y1="2.046" x2="13.5524" y2="2.046" width="0.254" layer="16"/>
+<wire x1="13.5524" y1="2.046" x2="12.4" y2="3.3" width="0.254" layer="16"/>
 <wire x1="12.4" y1="3.3" x2="6.7" y2="3.3" width="0.254" layer="16"/>
 <wire x1="6.7" y1="3.3" x2="4.5" y2="5.5" width="0.254" layer="16"/>
+<wire x1="24.5248" y1="2.9248" x2="23.646" y2="2.046" width="0.254" layer="1"/>
 </signal>
 <signal name="N$2">
@@
 <contactref element="U1" pad="9"/>
 <contactref element="U$6" pad="P$1"/>
-<wire x1="1.6016" y1="27.4956" x2="1.6016" y2="33.9214" width="1.016" layer="16"/>
-<wire x1="1.6016" y1="33.9214" x2="1.6268" y2="33.9466" width="1.016" layer="16"/>
+<wire x1="1.6016" y1="27.4956" x2="1.6016" y2="18.7212" width="1.016" layer="16"/>
+<wire x1="1.6016" y1="18.7212" x2="1.5748" y2="18.6944" width="1.016" layer="16"/>
+<via x="1.5748" y="18.6944" extent="1-16" drill="0.35" diameter="0.127"/>
+<wire x1="1.5748" y1="18.6944" x2="1.5748" y2="5.9946" width="1.016" layer="1"/>
+<wire x1="1.5748" y1="5.9946" x2="1.5268" y2="5.9466" width="1.016" layer="1"/>
 </signal>
 <signal name="N$3">
 <contactref element="DS3234" pad="16"/>
 <contactref element="BAT1" pad="PWR@1"/>
-<wire x1="6.5718" y1="8.035" x2="3.765" y2="8.035" width="0.254" layer="1"/>
-<wire x1="3.765" y1="8.035" x2="2.5" y2="9.3" width="0.254" layer="1"/>
-<wire x1="2.5" y1="17.2" x2="2.5" y2="9.3" width="0.254" layer="1"/>
-<wire x1="5.768" y1="18.4252" x2="3.7252" y2="18.4252" width="0.254" layer="1"/>
-<wire x1="3.7252" y1="18.4252" x2="2.5" y2="17.2" width="0.254" layer="1"/>
+<wire x1="6.5718" y1="8.035" x2="4.865" y2="8.035" width="0.254" layer="1"/>
+<wire x1="4.865" y1="8.035" x2="4.3" y2="8.6" width="0.254" layer="1"/>
+<wire x1="4.3" y1="15" x2="4.3" y2="8.6" width="0.254" layer="1"/>
+<wire x1="5.768" y1="18.4252" x2="5.768" y2="16.468" width="0.254" layer="1"/>
+<wire x1="5.768" y1="16.468" x2="4.3" y2="15" width="0.254" layer="1"/>
 </signal>
 <signal name="D7_SS">
